File: customDisplay.kicad_pcb (KiCad board)
At the start: 4 copper layers, 76.2 x 68.6 mm, 114 parts, among them J1 STDC14, J2 B2B_TOP, J3 B2B_TOP, J4 LCD, J5 TOUCH, J6 USB_B_Micro, J7 5V_IN, J8 STDC14_TAG, SW1 BOOT, SW2 RESET, U1 STM32F767BGTx, U2 MT48LC4M32B2TG, U3 TSC2007, U4 TPS61169, U5 MT25QL512ABB, U6 USBLC6-2SC6, U7 USBLC6-2SC6, U8 AMS1117-3.3, X1 32.768kHz, X2 25MHz

Commit message: Update to REV B1
Parts:
- removed the REF** at (154.4, 101.3)
- added REF**: KiCad-Logo2_20mm_SilkScreen, Symbol:KiCad-Logo2_20mm_SilkScreen, B.Cu at (153.0, 101.8)
- C23: footprint jlcpcb_smt:C_0603_1608Metric -> jlcpcb_smt:C_0805_2012Metric
- SW1: value BOOT -> TACT
- SW2: value RESET -> TACT
Routing:
- net GND: track 165.0 -> 163.8 mm
- net /MCU/SWO: track 104.8 -> 104.7 mm, vias 3 -> 2
Other:
- board text added: "REV B1"
- board text removed: "REV A0"
