File: mcu.sch (KiCad schematic (older format))
At the start: 44 parts, among them J1 STDC14, J2 B2B_TOP, J3 B2B_TOP, J8 STDC14_TAG, SW1 TACT, SW2 TACT, U1 STM32F767BGTx, X1 32.768kHz, X2 25MHz

Commit message: Update to REV B1
Parts:
- C23: footprint jlcpcb_smt:C_0603_1608Metric -> jlcpcb_smt:C_0805_2012Metric
Changed lines of the file:
@@
 encoding utf-8
 Sheet 2 7
-Title "MCU"
+Title "svcguy"
 Date "2020-09-17"
-Rev "A0"
-Comp "svcguy"
+Rev "B1"
+Comp "Checked by Andy"
 Comment1 "Checked by Andy"
 Comment2 ""
@@
 F 0 "C23" H 5165 3296 50  0000 L CNN
 F 1 "4.7uF" H 5165 3205 50  0000 L CNN
-F 2 "jlcpcb_smt:C_0603_1608Metric" H 5088 3100 50  0001 C CNN
+F 2 "jlcpcb_smt:C_0805_2012Metric" H 5088 3100 50  0001 C CNN
 F 3 "~" H 5050 3250 50  0001 C CNN
 F 4 "C19666" H 5050 3250 50  0001 C CNN "LCSC"
